File: pcb_rev4/v04_left.sch (KiCad schematic (older format))
At the start: 74 parts, among them SW1 SW_Push, U1 ProMicro

Commit message: Repositioned both thumb clusters; fixed positioning of z key on left side
Parts:
- MX45: footprint MX_Only:MXOnly-1.5U-NoLED -> MX_Only:MXOnly-2U-NoLED
Changed lines of the file:
@@
 F 0 "MX45" H 7483 4673 60  0000 C CNN
 F 1 "MX-NoLED" H 7483 4599 20  0000 C CNN
-F 2 "MX_Only:MXOnly-1.5U-NoLED" H 6825 4425 60  0001 C CNN
+F 2 "MX_Only:MXOnly-2U-NoLED" H 6825 4425 60  0001 C CNN
 F 3 "" H 6825 4425 60  0001 C CNN
 	1    7450 4450
