File: pcb/v2.0/bourbondox2_right.kicad_pcb (KiCad board)
At the start: 2 copper layers, 158.8 x 157.2 mm, 65 parts, among them J1 MJ-4PP-9, SW1 SW_Push, U1 ProMicro

Commit message: Cleaning files off Asus ZenBook
Other:
- net class Default removed
